Commit message: Fix joint_3 transformation

File: urdf/robot.urdf (robot description, URDF)
Before this commit: robot yaro_1115, 8 links, 7 joints
Joints:
- joint joint_3: origin xyz=0.00000000 -0.49000000 0.00000000 rpy=3.14159265 0.00000000 0.00000000 -> xyz=0.0000000000 -0.4650000000 -0.0011000000 rpy=-3.1415926536 0.0000000000 0.0000000000
